File: kicad/headamp2/headamp2.sch (KiCad schematic (older format))
At the start: 34 parts, among them J1 AudioJack3, Q1 MP21, Q10 MP38, Q2 MP21, Q3 MP21, Q4 MP21, Q5 MP38, Q6 MP21, Q7 MP21, Q8 MP21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

Commit message: additional schematics
Parts:
- added R15, R16: 1K, symbol Device:R
- Q1, Q10, Q2, Q3, Q4, Q5, Q6, Q7, Q8, Q9: footprint (none) -> Package_TO_SOT_THT:TO-8-3
Connections:
- net GND: now also R15.2, R16.2
- net at C4.1, J1.T: now also R15.1
- net at C8.1, J1.R: now also R16.1
Other:
- moved on the sheet: J1
Changed lines of the file:
@@
 F 0 "Q1" H 6640 2046 50  0000 L CNN
 F 1 "MP21" H 6640 1955 50  0000 L CNN
-F 2 "" H 6650 2100 50  0001 C CNN
+F 2 "Package_TO_SOT_THT:TO-8-3" H 6650 2100 50  0001 C CNN
 F 3 "~" H 6450 2000 50  0001 C CNN
 	1    6450 2000
@@
 F 0 "Q2" H 7790 1546 50  0000 L CNN
 F 1 "MP21" H 7790 1455 50  0000 L CNN
-F 2 "" H 7800 1600 50  0001 C CNN
+F 2 "Package_TO_SOT_THT:TO-8-3" H 7800 1600 50  0001 C CNN
 F 3 "~" H 7600 1500 50  0001 C CNN
 	1    7600 1500
@@
 F 0 "Q4" H 8240 1796 50  0000 L CNN
 F 1 "MP21" H 8240 1705 50  0000 L CNN
-F 2 "" H 8250 1850 50  0001 C CNN
+F 2 "Package_TO_SOT_THT:TO-8-3" H 8250 1850 50  0001 C CNN
 F 3 "~" H 8050 1750 50  0001 C CNN
 	1    8050 1750
@@
 F 0 "Q5" H 8240 2304 50  0000 L CNN
 F 1 "MP38" H 8240 2395 50  0000 L CNN
-F 2 "" H 8250 2450 50  0001 C CNN
+F 2 "Package_TO_SOT_THT:TO-8-3" H 8250 2450 50  0001 C CNN
 F 3 "~" H 8050 2350 50  0001 C CNN
 	1    8050 2350
@@
 Wire Wire Line
 	8150 2550 8150 2750
-Wire Wire Line
-	8150 2750 7900 2750
 Wire Wire Line
 	7700 2700 7700 2750
@@
 F 0 "Q3" H 7790 2196 50  0000 L CNN
 F 1 "MP21" H 7790 2105 50  0000 L CNN
-F 2 "" H 7800 2250 50  0001 C CNN
+F 2 "Package_TO_SOT_THT:TO-8-3" H 7800 2250 50  0001 C CNN
 F 3 "~" H 7600 2150 50  0001 C CNN
 	1    7600 2150
@@
 	7950 1000 7700 1000
 $Comp
-L power:PWR_FLAG #FLG0102
-U 1 1 60ABF994
-P 7900 2750
-F 0 "#FLG0102" H 7900 2825 50  0001 C CNN
-F 1 "PWR_FLAG" H 7900 2923 50  0001 C CNN
-F 2 "" H 7900 2750 50  0001 C CNN
-F 3 "~" H 7900 2750 50  0001 C CNN
-	1    7900 2750
-	1    0    0    1
-$EndComp
-Connection ~ 7900 2750
-Wire Wire Line
-	7900 2750 7700 2750
-$Comp
 L Device:R R9
 U 1 1 60AFD3F0
@@
 F 0 "Q6" H 6690 4396 50  0000 L CNN
 F 1 "MP21" H 6690 4305 50  0000 L CNN
-F 2 "" H 6700 4450 50  0001 C CNN
+F 2 "Package_TO_SOT_THT:TO-8-3" H 6700 4450 50  0001 C CNN
 F 3 "~" H 6500 4350 50  0001 C CNN
 	1    6500 4350
@@
 F 0 "Q7" H 7840 3896 50  0000 L CNN
 F 1 "MP21" H 7840 3805 50  0000 L CNN
-F 2 "" H 7850 3950 50  0001 C CNN
+F 2 "Package_TO_SOT_THT:TO-8-3" H 7850 3950 50  0001 C CNN
 F 3 "~" H 7650 3850 50  0001 C CNN
 	1    7650 3850
@@
 F 0 "Q9" H 8290 4146 50  0000 L CNN
 F 1 "MP21" H 8290 4055 50  0000 L CNN
-F 2 "" H 8300 4200 50  0001 C CNN
+F 2 "Package_TO_SOT_THT:TO-8-3" H 8300 4200 50  0001 C CNN
 F 3 "~" H 8100 4100 50  0001 C CNN
 	1    8100 4100
@@
 F 0 "Q10" H 8290 4654 50  0000 L CNN
 F 1 "MP38" H 8290 4745 50  0000 L CNN
-F 2 "" H 8300 4800 50  0001 C CNN
+F 2 "Package_TO_SOT_THT:TO-8-3" H 8300 4800 50  0001 C CNN
 F 3 "~" H 8100 4700 50  0001 C CNN
 	1    8100 4700
@@
 Wire Wire Line
 	8400 4350 8200 4350
-Wire Wire Line
-	8600 4350 8750 4350
 Connection ~ 6600 3350
 Connection ~ 7200 3350
@@
 F 0 "Q8" H 7840 4546 50  0000 L CNN
 F 1 "MP21" H 7840 4455 50  0000 L CNN
-F 2 "" H 7850 4600 50  0001 C CNN
+F 2 "Package_TO_SOT_THT:TO-8-3" H 7850 4600 50  0001 C CNN
 F 3 "~" H 7650 4500 50  0001 C CNN
 	1    7650 4500
@@
 $EndComp
 Connection ~ 8100 3350
-Wire Wire Line
-	8100 3350 8000 3350
-$Comp
-L power:PWR_FLAG #FLG02
-U 1 1 60AFD67E
-P 8000 3350
-F 0 "#FLG02" H 8000 3425 50  0001 C CNN
-F 1 "PWR_FLAG" H 8000 3523 50  0001 C CNN
-F 2 "" H 8000 3350 50  0001 C CNN
-F 3 "~" H 8000 3350 50  0001 C CNN
-	1    8000 3350
-	1    0    0    -1
-$EndComp
-Connection ~ 8000 3350
-Wire Wire Line
-	8000 3350 7750 3350
 $Comp
 L power:PWR_FLAG #FLG01
@@
 L Connector:AudioJack3 J1
 U 1 1 60B0966F
-P 9050 3150
-F 0 "J1" H 8770 3083 50  0000 R CNN
-F 1 "AudioJack3" H 8770 3174 50  0000 R CNN
-F 2 "" H 9050 3150 50  0001 C CNN
-F 3 "~" H 9050 3150 50  0001 C CNN
-	1    9050 3150
+P 9300 3150
+F 0 "J1" H 9020 3083 50  0000 R CNN
+F 1 "AudioJack3" H 9020 3174 50  0000 R CNN
+F 2 "" H 9300 3150 50  0001 C CNN
+F 3 "~" H 9300 3150 50  0001 C CNN
+	1    9300 3150
 	-1   0    0    1
 $EndComp
 Wire Wire Line
-	8850 3050 8750 3050
-Wire Wire Line
-	8750 3050 8750 2000
-Wire Wire Line
-	8600 2000 8750 2000
-Wire Wire Line
-	8850 3150 8750 3150
-Wire Wire Line
-	8750 3150 8750 4350
-Wire Wire Line
-	8850 3250 8850 3450
+	9100 3050 9000 3050
+Wire Wire Line
+	9000 3050 9000 2000
+Wire Wire Line
+	9100 3150 9000 3150
+Wire Wire Line
+	9000 3150 9000 4350
+Wire Wire Line
+	9100 3250 9100 3450
 $Comp
 L power:GND #PWR07
 U 1 1 60B152BE
-P 8850 3450
-F 0 "#PWR07" H 8850 3200 50  0001 C CNN
-F 1 "GND" H 8855 3277 50  0000 C CNN
-F 2 "" H 8850 3450 50  0001 C CNN
-F 3 "" H 8850 3450 50  0001 C CNN
-	1    8850 3450
+P 9100 3450
+F 0 "#PWR07" H 9100 3200 50  0001 C CNN
+F 1 "GND" H 9105 3277 50  0000 C CNN
+F 2 "" H 9100 3450 50  0001 C CNN
+F 3 "" H 9100 3450 50  0001 C CNN
+	1    9100 3450
 	1    0    0    -1
 $EndComp
@@
 	1    0    0    -1
 $EndComp
+Wire Wire Line
+	8600 2000 8800 2000
+Wire Wire Line
+	8600 4350 8800 4350
+$Comp
+L Device:R R16
+U 1 1 60B283C7
+P 8800 4900
+F 0 "R16" H 8870 4946 50  0000 L CNN
+F 1 "1K" H 8870 4855 50  0000 L CNN
+F 2 "" V 8730 4900 50  0001 C CNN
+F 3 "~" H 8800 4900 50  0001 C CNN
+	1    8800 4900
+	1    0    0    -1
+$EndComp
+Wire Wire Line
+	8800 4750 8800 4350
+Connection ~ 8800 4350
+Wire Wire Line
+	8800 4350 9000 4350
+Wire Wire Line
+	8800 5050 8800 5100
+Wire Wire Line
+	8800 5100 8200 5100
+Connection ~ 8200 5100
+$Comp
+L Device:R R15
+U 1 1 60B2E7BA
+P 8800 2550
+F 0 "R15" H 8870 2596 50  0000 L CNN
+F 1 "1K" H 8870 2505 50  0000 L CNN
+F 2 "" V 8730 2550 50  0001 C CNN
+F 3 "~" H 8800 2550 50  0001 C CNN
+	1    8800 2550
+	1    0    0    -1
+$EndComp
+Wire Wire Line
+	8800 2400 8800 2000
+Connection ~ 8800 2000
+Wire Wire Line
+	8800 2000 9000 2000
+Wire Wire Line
+	8800 2700 8800 2750
+Wire Wire Line
+	8800 2750 8150 2750
+Connection ~ 8150 2750
+Wire Wire Line
+	7700 2750 8150 2750
+Wire Wire Line
+	7750 3350 8100 3350
 $EndSCHEMATC
