File: kicad/headamp2/_autosave-headamp2.sch (KiCad schematic (older format))
At the start: 30 parts, among them J1 AudioJack3, Q1 MP21, Q2 MP21, Q3 MP21, Q4 MP21, Q5 MP38, Q6 MP21, Q7 MP21

Commit message: mods
Signed-off-by: Badscrew <badscrew@dolganoff.com>
Parts:
- Q1, Q2: value MP21 -> MP39B
Changed lines of the file:
@@
 P 6000 2000
 F 0 "Q2" H 6190 2046 50  0000 L CNN
-F 1 "MP21" H 6190 1955 50  0000 L CNN
+F 1 "MP39B" H 6190 1955 50  0000 L CNN
 F 2 "Package_TO_SOT_THT:TO-8-3" H 6200 2100 50  0001 C CNN
 F 3 "~" H 6000 2000 50  0001 C CNN
@@
 U 1 1 60A9DE5E
 P 5550 2000
-F 0 "C3" V 5775 2000 50  0000 C CNN
-F 1 "10uF" V 5684 2000 50  0000 C CNN
+F 0 "C3" V 5400 2000 50  0000 C CNN
+F 1 "10uF" V 5300 2000 50  0000 C CNN
 F 2 "" H 5550 2000 50  0001 C CNN
 F 3 "~" H 5550 2000 50  0001 C CNN
@@
 P 4850 2000
 F 0 "Q1" H 5040 2046 50  0000 L CNN
-F 1 "MP21" H 5040 1955 50  0000 L CNN
+F 1 "MP39B" H 5040 1955 50  0000 L CNN
 F 2 "Package_TO_SOT_THT:TO-8-3" H 5050 2100 50  0001 C CNN
 F 3 "~" H 4850 2000 50  0001 C CNN
